File: first_project/first_project.kicad_pcb (KiCad board)
At the start: 2 copper layers, 140 x 90 mm, 4 parts

Commit message: updated with pcb
Parts:
- added BT1: Battery_Cell, footprints:BatteryHolder_Keystone_106_1x20mm, F.Cu at (154.9, 88.9)
- added C1: CP (1uF), footprints:C_0805_2012Metric, F.Cu at (163.4, 118.9)
- added C2: C (0.1uF), footprints:C_0805_2012Metric, F.Cu at (165.8, 115.9)
- added C3: 22pf, footprints:C_0805_2012Metric, F.Cu at (159.0, 118.9)
- added C4: C(0.1uF), footprints:C_0805_2012Metric, F.Cu at (142.5, 133.3)
- added C5: 22pf, footprints:C_0805_2012Metric, F.Cu at (154.6, 124.8)
- added C6: C_0805_0.1uf, footprints:C_0805_2012Metric, F.Cu at (198.5, 77.5)
- added C7: C(0.1uf), footprints:C_0805_2012Metric, F.Cu at (198.4, 80.6)
- added C8: C_0805_0.1uf, footprints:C_0805_2012Metric, F.Cu at (146.9, 133.3)
- added C9: C_0805_0.1uf, footprints:C_0805_2012Metric, F.Cu at (173.0, 103.2)
- added D1: LED, footprints:LED_0805_2012Metric, F.Cu at (129.2, 132.1)
- added D2: LED_0805_GRN, footprints:LED_0805_2012Metric, F.Cu at (122.7, 135.0)
- added D3: LED_0805_GRN, footprints:LED_0805_2012Metric, F.Cu at (194.1, 77.6)
- added D4: LED_0805_GRN, footprints:LED_0805_2012Metric, F.Cu at (127.1, 135.1)
- added D5: LED_0805_GRN, footprints:LED_0805_2012Metric, F.Cu at (137.3, 121.6)
- added D6: LED_0805_GRN, footprints:LED_0805_2012Metric, F.Cu at (148.5, 125.5)
- added D7: LED_0805_GRN, footprints:LED_0805_2012Metric, F.Cu at (138.1, 133.3)
- added D8: LED_0805_GRN, footprints:LED_0805_2012Metric, F.Cu at (133.7, 133.3)
- added DS1: LED_Display_1001, footprints:Adafruit-1001-0-0-MFG, F.Cu at (120.2, 101.9)
- added J1: Conn_01x06, footprints:PinHeader_1x06_P2.54mm_Vertical, F.Cu at (132.7, 115.5)
- added J2: PJ-102AH, footprints:PJ-102AH, F.Cu at (147.3, 118.9)
- added J3: Conn_02x03_Odd_Even, footprints:PinHeader_2x03_P2.54mm_Vertical, F.Cu at (165.9, 104.1)
- added R1: 2.2K, footprints:R_0805_2012Metric, F.Cu at (154.6, 121.9)
- added R10: R_0805_22K, footprints:R_0805_2012Metric, F.Cu at (194.4, 86.5)
- added R11: R_0805_10K, footprints:R_0805_2012Metric, F.Cu at (165.8, 112.9)
- added R12: R_0805_10K, footprints:R_0805_2012Metric, F.Cu at (148.5, 128.5)
- added R2: 10K, footprints:R_0805_2012Metric, F.Cu at (183.2, 97.1)
- added R3: R_0805_4.7K, footprints:R_0805_2012Metric, F.Cu at (170.2, 112.9)
- added R4: R_0805_4.7K, footprints:R_0805_2012Metric, F.Cu at (154.6, 118.9)
- added R5: R_0805_10K, footprints:R_0805_2012Metric, F.Cu at (173.0, 106.2)
- added R6: R_0805_10K, footprints:R_0805_2012Metric, F.Cu at (159.0, 121.9)
- added R7: R_0805_10K, footprints:R_0805_2012Metric, F.Cu at (152.9, 128.5)
- added R8: R_0805_10K, footprints:R_0805_2012Metric, F.Cu at (194.0, 80.6)
- added R9: R_0805_10K, footprints:R_0805_2012Metric, F.Cu at (194.0, 83.5)
- added SW1: Omron_B3F_SPST, footprints:SW_SPST_Omron_B3FS-100xP, F.Cu at (158.0, 113.5)
- added SW2: Omron_B3F_SPST, footprints:SW_SPST_Omron_B3FS-100xP, F.Cu at (140.7, 127.9)
- added SW3: Omron_B3F_SPST, footprints:SW_SPST_Omron_B3FS-100xP, F.Cu at (114.9, 131.6)
- added SW4: Omron_B3F_SPST, footprints:SW_SPST_Omron_B3FS-100xP, F.Cu at (158.0, 105.7)
- added SW5: Omron_B3F_SPST, footprints:SW_SPST_Omron_B3FS-100xP, F.Cu at (186.6, 91.7)
- added U1: ATmega328-PU, footprints:DIP-28_W7.62mm, F.Cu at (132.0, 78.1)
- added U2: L7805_TO92, footprints:TO-92_Inline, F.Cu at (122.4, 131.0)
- added U3: DS1307_DIP-8, footprints:DIP-8_W7.62mm, F.Cu at (182.6, 78.1)
- added U4: MAX7219, footprints:DIP-24_W7.62mm, F.Cu at (142.9, 78.1)
- added Y1: Crystal(16MHz), footprints:Crystal_SMD_2Pin_3.2x1.5mm, F.Cu at (137.6, 114.9)
- added Y2: Crystal_32768Hz, footprints:Crystal_SMD_2Pin_3.2x1.5mm, F.Cu at (137.6, 118.4)

Commit message: pcb routing
Parts:
- removed R6, R7, R8: R_0805_10K, footprints:R_0805_2012Metric
- added R13: R_0805_4.7K, footprints:R_0805_2012Metric, F.Cu at (142.2, 61.0)
- added R14: R_0805_4.7K, footprints:R_0805_2012Metric, F.Cu at (137.2, 61.0)
- J2: value PJ-102AH -> Power_inlet_vertical; footprint footprints:PJ-102AH -> footprints:Wurth-694106402002
- U2: footprint footprints:TO-92_Inline -> footprints:TO-252-2
- moved R9 78.2 mm to (137.2, 137.2)
- moved J1 72.1 mm to (198.1, 85.1)
- moved U2 69.0 mm to (190.5, 119.4)
- moved R5 68.6 mm to (111.8, 137.2)
- moved U3 64.3 mm to (120.7, 61.0)
- moved R1 61.1 mm to (94.0, 129.5)
- moved Y2 60.8 mm to (114.3, 62.2)
- moved D3 60.3 mm to (134.6, 87.3)
- moved D8 59.8 mm to (171.8, 87.3)
- moved SW1 58.3 mm to (210.8, 88.9)
- moved C2 57.2 mm to (149.9, 61.0), turned to 180 degrees
- moved C4 54.9 mm to (193.0, 111.8)
- moved D7 53.4 mm to (165.1, 87.3)
- moved R2 52.9 mm to (134.6, 76.2), turned to 90 degrees
- moved R3 51.5 mm to (210.8, 81.3)
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Connections:
- net Net-(D2-Pad1) renamed /DIG_5
- net Net-(R10-Pad2) renamed /ISET
Routing:
- net /DIG_5: track 0.00 -> 116.3 mm
- net /SEG_G: track 0.00 -> 53.2 mm, vias 0 -> 2
- net /SEG_C: track 0.00 -> 44.6 mm, vias 0 -> 1
- net GND: track 0.00 -> 35.6 mm, vias 0 -> 2
- net Net-(C1-Pad1): track 0.00 -> 34.8 mm
- net SDA_RTC: track 0.00 -> 28.1 mm, vias 0 -> 1
- net MOSI: track 0.00 -> 27.2 mm, vias 0 -> 2
- net /SEG_D: track 0.00 -> 25.5 mm, vias 0 -> 2
- net /SEG_B: track 0.00 -> 24.5 mm
- net MISO: track 0.00 -> 22.9 mm
- net /SEG_F: track 0.00 -> 22.0 mm, vias 0 -> 1
- net /SEG_A: track 0.00 -> 18.9 mm
- net /DIG_3: track 0.00 -> 17.6 mm
- net Net-(BT1-Pad1): track 0.00 -> 14.7 mm
- net SCL_RTC: track 0.00 -> 13.6 mm
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- added copper zone on B.Cu, net GND
- added copper zone on F.Cu, net VCC

Commit message: first fully connected pcb. very terrible
Parts:
- U2: moved to B.Cu
- moved R1 7.73 mm to (101.6, 128.3)
- moved R3 3.81 mm to (207.0, 81.3)
- moved SW1 3.81 mm to (207.0, 88.9)
- moved C6 3.81 mm to (207.9, 96.5)
- moved D1 2.54 mm to (101.6, 132.1)
- moved C8 1.27 mm to (172.7, 124.5)
- moved J1 1.27 mm to (196.8, 85.1)
- turned U2 to 180 degrees
Routing:
- net BTN_MIN: track 0.00 -> 189.3 mm
- net LED_SCK: track 0.00 -> 164.7 mm
- net RESET: track 2.97 -> 144.5 mm, vias 0 -> 1
- net DISP_LOAD: track 0.00 -> 125.9 mm, vias 0 -> 1
- net DISP_DATA: track 0.00 -> 118.6 mm
- net BTN_HOUR: track 0.00 -> 114.3 mm, vias 0 -> 1
- net GND: track 35.6 -> 148.7 mm, vias 2 -> 1
- net BTN_SETOPT: track 0.00 -> 107.8 mm, vias 0 -> 1
- net RXD: track 0.00 -> 88.9 mm, vias 0 -> 2
- net BTN_DAY: track 0.00 -> 80.7 mm
- net /SEG_F: track 22.0 -> 96.3 mm, vias 1 -> 2
- net DISP_CLK: track 0.00 -> 69.6 mm
- net /SEG_B: track 24.5 -> 92.4 mm, vias 0 -> 2
- net /DIG_0: track 0.00 -> 57.5 mm
- net TXD: track 0.00 -> 56.4 mm, vias 0 -> 2
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
Commit message: updated
Routing:
- net BTN_HOUR: track 114.3 -> 119.8 mm, vias 1 -> 2
- net Net-(C6-Pad2): track 18.0 -> 12.5 mm
- net /XTAL1: track 9.98 -> 14.5 mm, vias 1 -> 2
- net Net-(J1-Pad4): track 2.96 -> 7.08 mm
- net GND: track 148.7 -> 145.4 mm, vias 1 -> 2
- net /SEG_DP: track 37.9 -> 34.9 mm
- net DISP_LOAD: track 125.9 -> 124.1 mm
- net RESET: track 144.5 -> 145.9 mm, vias 1 -> 2
- net BTN_DAY: track 80.7 -> 81.5 mm
- net Net-(C1-Pad1): track 40.7 -> 41.1 mm, vias 0 -> 1
- net TXD: track 56.4 -> 56.8 mm, vias 2 -> 3
- net RXD: track 88.9 -> 89.3 mm, vias 2 -> 3
- net BTN_MIN: track 189.3 -> 189.6 mm, vias 0 -> 1
- net BTN_SETOPT: vias 1 -> 2

Commit message: new routing + gerber
Parts:
- J2: moved to B.Cu
- U2: value L7805_TO92 -> L7805; moved to F.Cu
- moved D1 75.2 mm to (129.5, 62.2)
- moved R1 65.3 mm to (130.8, 69.8), turned to 180 degrees
- moved R12 61.0 mm to (176.1, 76.2), turned to 180 degrees
- moved R5 58.7 mm to (133.3, 82.5)
- moved R9 55.5 mm to (147.3, 82.5)
- moved R11 54.9 mm to (163.4, 82.5)
- moved C9 50.8 mm to (127.6, 104.8)
- moved SW2 49.9 mm to (137.2, 88.9), turned to 180 degrees
- moved SW3 48.5 mm to (152.4, 88.9), turned to 180 degrees
- moved SW5 48.3 mm to (182.9, 88.9), turned to 180 degrees
- moved SW4 48.3 mm to (167.6, 88.9), turned to 180 degrees
- moved C8 48.2 mm to (127.4, 108.0)
- moved D8 46.8 mm to (180.3, 133.3)
- moved D2 46.7 mm to (134.6, 133.3)
- moved D3 46.7 mm to (142.2, 133.3)
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Connections:
- U2 pad 1: VCC -> Net-(C1-Pad1)
- U2 pad 3: Net-(C1-Pad1) -> VCC
Routing:
- net /SEG_E: track 48.0 -> 237.9 mm, vias 1 -> 2
- net BTN_MIN: track 189.6 -> 24.5 mm, vias 1 -> 0
- net BTN_HOUR: track 119.8 -> 23.3 mm, vias 2 -> 0
- net DISP_CLK: track 69.6 -> 166.1 mm, vias 0 -> 1
- net LED_SCK: track 164.7 -> 68.7 mm, vias 0 -> 2
- net BTN_SETOPT: track 107.8 -> 30.1 mm, vias 2 -> 0
- net GND: track 145.4 -> 214.8 mm, vias 2 -> 3
- net /DIG_3: track 17.6 -> 81.0 mm, vias 0 -> 3
- net /SEG_C: track 44.6 -> 104.3 mm
- net BTN_DAY: track 81.5 -> 32.3 mm
- net DISP_DATA: track 118.6 -> 69.6 mm
- net /DIG_4: track 33.7 -> 81.3 mm
- net /SEG_D: track 40.0 -> 81.7 mm, vias 2 -> 1
- net Net-(J1-Pad5): track 54.1 -> 15.9 mm
- net RESET: track 145.9 -> 108.6 mm
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Other:
- board text added: "Lovely_Clock"

Commit message: final. I hope
Parts:
- added TP1: TestPoint, footprints:TestPoint_THTPad_D2.0mm_Drill1.0mm, F.Cu at (193.0, 113.0)
- added TP2: TestPoint, footprints:TestPoint_THTPad_D2.0mm_Drill1.0mm, F.Cu at (124.5, 85.1)
- added TP3: TestPoint, footprints:TestPoint_THTPad_D2.0mm_Drill1.0mm, F.Cu at (123.2, 61.0)
- added TP4: TestPoint, footprints:TestPoint_THTPad_D2.0mm_Drill1.0mm, F.Cu at (104.1, 61.0)
- added TP5: TestPoint, footprints:TestPoint_THTPad_D2.0mm_Drill1.0mm, F.Cu at (108.0, 106.7)
- added TP6: TestPoint, footprints:TestPoint_THTPad_D2.0mm_Drill1.0mm, F.Cu at (158.8, 81.3)
- added TP7: TestPoint, footprints:TestPoint_THTPad_D2.0mm_Drill1.0mm, F.Cu at (96.5, 115.6)
Routing:
- net VCC: track 26.6 -> 65.2 mm, vias 3 -> 8
- net SCL_RTC: track 26.4 -> 40.0 mm
- net DISP_CLK: track 166.1 -> 177.1 mm
- net SDA_RTC: track 26.6 -> 37.3 mm
- net DISP_LOAD: track 97.1 -> 102.7 mm
- net Net-(BT1-Pad1): track 25.0 -> 30.1 mm
- net DISP_DATA: track 69.6 -> 72.7 mm

Commit message: final gerber hopefully
Parts:
- moved TP6 41.9 mm to (116.8, 82.5)
- moved C3 16.9 mm to (160.0, 61.4), turned to -90 degrees
- moved TP7 9.92 mm to (104.1, 121.9)
- moved TP5 3.81 mm to (108.0, 110.5)
- moved TP2 2.84 mm to (123.2, 82.5)
- moved TP4 2.54 mm to (104.1, 63.5)
- moved R10 1.81 mm to (125.7, 111.1), turned to -90 degrees
Routing:
- net /DIG_2: track 46.9 -> 140.5 mm, vias 0 -> 2
- net GND: track 214.8 -> 168.0 mm, vias 3 -> 13
- net DISP_LOAD: track 102.7 -> 91.2 mm
- net /XTAL1: track 8.06 -> 18.4 mm, vias 0 -> 1
- net DISP_CLK: track 177.1 -> 167.9 mm
- net VCC: track 65.2 -> 57.8 mm, vias 8 -> 7
- net /DIG_3: track 81.0 -> 75.5 mm
- net MISO: track 22.9 -> 19.3 mm
- net Net-(C1-Pad1): track 64.4 -> 67.8 mm
- net /SEG_A: track 73.5 -> 70.4 mm
- net SDA_RTC: track 37.3 -> 34.2 mm
- net /SEG_F: track 115.2 -> 112.2 mm
- net Net-(BT1-Pad1): track 30.1 -> 27.6 mm
- net /DIG_4: track 81.3 -> 79.1 mm
- net /SEG_E: track 237.9 -> 235.9 mm
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
Commit message: new changes
Parts:
- removed R13, R14: R_0805_4.7K, footprints:R_0805_2012Metric
- added R6: R_0805_4.7K, footprints:R_0805_2012Metric, F.Cu at (143.5, 62.2)
- added R7: R_0805_4.7K, footprints:R_0805_2012Metric, F.Cu at (138.4, 61.0)
- C1: value CP (1uF) -> C_0805_1uf
- C2: value C (0.1uF) -> C_0805_0.1uf
- C3, C5: value 22pf -> C_0805_22pf
- C4: value C(0.1uF) -> C_0805_0.1uf
- C7: value C(0.1uf) -> C_0805_0.1uf
- C8: value C_0805_0.1uf -> C_0805_10uf
- D1: value LED -> LED_0805
- R1: value 2.2K -> R_0805_2.2K
- R2: value 10K -> R_0805_10K
- Y1: value Crystal(16MHz) -> Crystal_32768Hz
- moved C7 74.6 mm to (201.9, 128.3)
- moved C4 59.4 mm to (153.7, 76.2)
- moved C1 33.5 mm to (203.6, 95.2)
- moved C8 0.42 mm to (127.0, 108.0)
Connections:
- C7 pad 2: Net-(C7-Pad2) -> GND
- U1 pad 20: Net-(C7-Pad2) -> VCC
- U1 pad 26: SDA_RTC -> unconnected-(U1-Pad26)
- U1 pad 27: SCL_RTC -> SDA_RTC
- U1 pad 28: unconnected-(U1-Pad28) -> SCL_RTC
- U1 pad 7: Net-(C7-Pad2) -> VCC
Routing:
- net VCC: track 57.8 -> 30.0 mm, vias 7 -> 1
- net Net-(C7-Pad2): track 17.3 -> 0.00 mm, vias 1 -> 0
- net GND: track 168.0 -> 172.5 mm, vias 13 -> 14
- net Net-(C1-Pad1): track 67.8 -> 72.0 mm
