File: first_project/first_project.kicad_sch (KiCad schematic)
At the start: 21 parts, among them J1 Conn_01x06, J2 PJ-102AH, SW1 Omron_B3F_SPST, U1 ATmega328-PU, U2 L7805_TO92, Y1 Crystal

Commit message: Schematic update
Parts:
- added C7: C(0.1uf), footprints:C_0805_2012Metric, symbol HPS:C_0805_0.1uf
- C1: value CP -> CP (1uF)
- C2: value C -> C (0.1uF)
- C4: value C -> C(0.1uF)
- Y1: value Crystal -> Crystal(16MHz)
Connections:
- net VCC: now also C7.1; no longer U1.20 (AVCC), U1.7 (VCC)
- new net: C7.2, U1.20 (AVCC), U1.7 (VCC)
Changed lines of the file:
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@@
   (junction (at 201.93 74.93) (diameter 0) (color 0 0 0 0)
   )
+  (junction (at 115.57 27.94) (diameter 0) (color 0 0 0 0)
+  )
   (junction (at 330.2 54.61) (diameter 0) (color 0 0 0 0)
   )
   (junction (at 341.63 44.45) (diameter 0) (color 0 0 0 0)
-  )
-  (junction (at 115.57 25.4) (diameter 0) (color 0 0 0 0)
   )
   (junction (at 182.88 149.86) (diameter 0) (color 0 0 0 0)
@@
     (stroke (width 0) (type default) (color 0 0 0 0))
   )
+  (wire (pts (xy 115.57 27.94) (xy 118.11 27.94))
+    (stroke (width 0) (type default) (color 0 0 0 0))
+  )
   (polyline (pts (xy 76.2 13.97) (xy 237.49 13.97))
     (stroke (width 0) (type default) (color 0 0 0 0))
   )
+  (wire (pts (xy 115.57 27.94) (xy 115.57 29.21))
+    (stroke (width 0) (type default) (color 0 0 0 0))
+  )
   (polyline (pts (xy 278.13 17.78) (xy 278.13 67.31))
     (stroke (width 0) (type default) (color 0 0 0 0))
@@
     (stroke (width 0) (type default) (color 0 0 0 0))
   )
+  (wire (pts (xy 118.11 29.21) (xy 118.11 27.94))
+    (stroke (width 0) (type default) (color 0 0 0 0))
+  )
   (polyline (pts (xy 101.6 134.62) (xy 129.54 134.62))
     (stroke (width 0) (type default) (color 0 0 0 0))
@@
     (stroke (width 0) (type default) (color 0 0 0 0))
   )
-  (wire (pts (xy 118.11 25.4) (xy 115.57 25.4))
-    (stroke (width 0) (type default) (color 0 0 0 0))
-  )
   (wire (pts (xy 115.57 149.86) (xy 115.57 152.4))
     (stroke (width 0) (type default) (color 0 0 0 0))
@@
     (stroke (width 0) (type default) (color 0 0 0 0))
   )
-  (wire (pts (xy 115.57 25.4) (xy 115.57 29.21))
-    (stroke (width 0) (type default) (color 0 0 0 0))
-  )
   (wire (pts (xy 175.26 149.86) (xy 182.88 149.86))
     (stroke (width 0) (type default) (color 0 0 0 0))
@@
     (stroke (width 0) (type default) (color 0 0 0 0))
   )
-  (wire (pts (xy 118.11 29.21) (xy 118.11 25.4))
-    (stroke (width 0) (type default) (color 0 0 0 0))
-  )
-  (wire (pts (xy 115.57 24.13) (xy 115.57 25.4))
-    (stroke (width 0) (type default) (color 0 0 0 0))
-  )
   (wire (pts (xy 201.93 71.12) (xy 201.93 74.93))
     (stroke (width 0) (type default) (color 0 0 0 0))
@@
   )
   (polyline (pts (xy 157.48 172.72) (xy 157.48 139.7))
+    (stroke (width 0) (type default) (color 0 0 0 0))
+  )
+  (wire (pts (xy 115.57 26.67) (xy 115.57 27.94))
     (stroke (width 0) (type default) (color 0 0 0 0))
   )
@@
       (effects (font (size 1.27 1.27)) (justify left))
     )
-    (property "Value" "CP" (id 1) (at 318.77 52.0699 0)
+    (property "Value" "CP (1uF)" (id 1) (at 318.77 52.0699 0)
       (effects (font (size 1.27 1.27)) (justify left))
     )
@@
   )
   (symbol (lib_id "HPS:Crystal_32768Hz") (at 158.75 44.45 90) (unit 1)
-    (in_bom yes) (on_board yes) (fields_autoplaced)
-    (property "Reference" "Y1" (id 0) (at 162.56 43.1799 90)
+    (in_bom yes) (on_board yes)
+    (property "Reference" "Y1" (id 0) (at 157.48 33.02 90)
       (effects (font (size 1.27 1.27)) (justify right))
     )
-    (property "Value" "Crystal" (id 1) (at 162.56 45.7199 90)
+    (property "Value" "Crystal(16MHz)" (id 1) (at 153.67 36.83 90)
       (effects (font (size 1.27 1.27)) (justify right))
     )
@@
       (effects (font (size 1.27 1.27)) (justify left))
     )
-    (property "Value" "C" (id 1) (at 87.63 45.72 0)
+    (property "Value" "C (0.1uF)" (id 1) (at 85.09 45.72 0)
       (effects (font (size 1.27 1.27)) (justify left))
     )
@@
     (pin "2")
   )
-  (symbol (lib_id "HPS:VCC") (at 115.57 24.13 0) (unit 1)
-    (in_bom yes) (on_board yes) (fields_autoplaced)
-    (property "Reference" "#PWR03" (id 0) (at 115.57 27.94 0)
-      (effects (font (size 1.27 1.27)) hide)
-    )
-    (property "Value" "VCC" (id 1) (at 115.57 19.05 0))
-    (property "Footprint" "" (id 2) (at 115.57 24.13 0)
-      (effects (font (size 1.27 1.27)) hide)
-    )
-    (property "Datasheet" "" (id 3) (at 115.57 24.13 0)
+  (symbol (lib_id "HPS:VCC") (at 115.57 19.05 0) (unit 1)
+    (in_bom yes) (on_board yes)
+    (property "Reference" "#PWR03" (id 0) (at 115.57 22.86 0)
+      (effects (font (size 1.27 1.27)) hide)
+    )
+    (property "Value" "VCC" (id 1) (at 120.65 16.51 0))
+    (property "Footprint" "" (id 2) (at 115.57 19.05 0)
+      (effects (font (size 1.27 1.27)) hide)
+    )
+    (property "Datasheet" "" (id 3) (at 115.57 19.05 0)
       (effects (font (size 1.27 1.27)) hide)
     )
@@
     )
     (pin "1")
+  )
+  (symbol (lib_id "HPS:C_0805_0.1uf") (at 115.57 22.86 0) (unit 1)
+    (in_bom yes) (on_board yes) (fields_autoplaced)
+    (property "Reference" "C7" (id 0) (at 119.38 21.5899 0)
+      (effects (font (size 1.27 1.27)) (justify left))
+    )
+    (property "Value" "C(0.1uf)" (id 1) (at 119.38 24.1299 0)
+      (effects (font (size 1.27 1.27)) (justify left))
+    )
+    (property "Footprint" "footprints:C_0805_2012Metric" (id 2) (at 116.5352 26.67 0)
+      (effects (font (size 1.27 1.27)) hide)
+    )
+    (property "Datasheet" "https://datasheets.avx.com/X7RDielectric.pdf" (id 3) (at 116.205 20.32 0)
+      (effects (font (size 1.27 1.27)) hide)
+    )
+    (property "MFG" "AVX Corporation" (id 4) (at 115.57 29.21 0)
+      (effects (font (size 1.27 1.27)) hide)
+    )
+    (property "MPN" "08055C104KAT2A" (id 5) (at 115.57 31.75 0)
+      (effects (font (size 1.27 1.27)) hide)
+    )
+    (property "Digikey PN" "478-1395-1-ND" (id 6) (at 115.57 36.83 0)
+      (effects (font (size 1.27 1.27)) hide)
+    )
+    (property "Mouser PN" "N/A" (id 7) (at 115.57 39.37 0)
+      (effects (font (size 1.27 1.27)) hide)
+    )
+    (property "Voltage" "N/A" (id 8) (at 115.57 41.91 0)
+      (effects (font (size 1.27 1.27)) hide)
+    )
+    (property "Dielectric" "N/A" (id 9) (at 115.57 41.91 0)
+      (effects (font (size 1.27 1.27)) hide)
+    )
+    (property "Tolerance" "N/A" (id 10) (at 115.57 41.91 0)
+      (effects (font (size 1.27 1.27)) hide)
+    )
+    (pin "1")
+    (pin "2")
   )
   (symbol (lib_id "HPS:R_0805_4.7K") (at 214.63 154.94 90) (unit 1)
@@
       (effects (font (size 1.27 1.27)) (justify left))
     )
-    (property "Value" "C" (id 1) (at 345.44 49.5299 0)
+    (property "Value" "C(0.1uF)" (id 1) (at 345.44 49.5299 0)
       (effects (font (size 1.27 1.27)) (justify left))
     )
@@
     )
     (path "/63fe69fa-19f2-4018-bfe2-85b6913817f2"
-      (reference "C1") (unit 1) (value "CP") (footprint "footprints:C_0805_2012Metric")
+      (reference "C1") (unit 1) (value "CP (1uF)") (footprint "footprints:C_0805_2012Metric")
     )
     (path "/6a193e0e-f417-4e70-afe6-70c1ec276b62"
-      (reference "C2") (unit 1) (value "C") (footprint "footprints:C_0805_2012Metric")
+      (reference "C2") (unit 1) (value "C (0.1uF)") (footprint "footprints:C_0805_2012Metric")
     )
     (path "/9e18c6c5-49cd-42dd-8bf2-5c8a36f8b156"
@@
     )
     (path "/d8ab444e-b777-418e-ac8e-74bcf0443e4e"
-      (reference "C4") (unit 1) (value "C") (footprint "footprints:C_0805_2012Metric")
+      (reference "C4") (unit 1) (value "C(0.1uF)") (footprint "footprints:C_0805_2012Metric")
     )
     (path "/9f67bbea-90ed-4ac8-9342-2215b3cadb97"
@@
       (reference "C6") (unit 1) (value "C_0805_0.1uf") (footprint "footprints:C_0805_2012Metric")
     )
+    (path "/c7869aba-7c1d-4121-b45f-5117350b0d3b"
+      (reference "C7") (unit 1) (value "C(0.1uf)") (footprint "footprints:C_0805_2012Metric")
+    )
     (path "/f1a32e71-1c04-4b5b-abef-668d7d3322a4"
       (reference "D1") (unit 1) (value "LED") (footprint "footprints:LED_0805_2012Metric")
@@
     )
     (path "/6442dc18-36db-40d9-883c-94941bf3bbe3"
-      (reference "Y1") (unit 1) (value "Crystal") (footprint "footprints:Crystal_SMD_2Pin_3.2x1.5mm")
-    )
-  )
+      (reference "Y1") (unit 1) (value "Crystal(16MHz)") (footprint "footprints:Crystal_SMD_2Pin_3.2x1.5mm")
+    )
+  )

Commit message: New file
Parts:
- added U?: DS1307_DIP-8, footprints:DIP-8_W7.62mm, symbol HPS:DS1307_DIP-8
Connections:
- net GND: now also U?.4 (GND)
- net VCC: now also U?.8 (VCC)
- net SDA_RTC: now reaches U1.26 (PC3)
- net SDA_RTC: now also U?.5 (SDA)
- net SCL_RTC: now reaches U1.27 (PC4)
- net SCL_RTC: now also U?.6 (SCL)
- new net +BATT: U?.3 (VBAT)
Other:
- note added: "RTC MODULE"
Changed lines of the file:
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@@
+    (stroke (width 0) (type default) (color 0 0 0 0))
+  )
+  (polyline (pts (xy 342.9 139.7) (xy 267.97 139.7))
     (stroke (width 0) (type default) (color 0 0 0 0))
   )
@@
     (stroke (width 0) (type default) (color 0 0 0 0))
   )
+  (wire (pts (xy 313.69 104.14) (xy 313.69 106.68))
+    (stroke (width 0) (type default) (color 0 0 0 0))
+  )
+  (wire (pts (xy 288.29 114.3) (xy 303.53 114.3))
+    (stroke (width 0) (type default) (color 0 0 0 0))
+  )
   (wire (pts (xy 100.33 36.83) (xy 96.52 36.83))
     (stroke (width 0) (type default) (color 0 0 0 0))
@@
     (stroke (width 0) (type default) (color 0 0 0 0))
   )
+  (wire (pts (xy 130.81 69.85) (xy 138.43 69.85))
+    (stroke (width 0) (type default) (color 0 0 0 0))
+  )
+  (wire (pts (xy 130.81 67.31) (xy 137.16 67.31))
+    (stroke (width 0) (type default) (color 0 0 0 0))
+  )
   (polyline (pts (xy 278.13 17.78) (xy 278.13 67.31))
     (stroke (width 0) (type default) (color 0 0 0 0))
   )
+  (wire (pts (xy 298.45 111.76) (xy 303.53 111.76))
+    (stroke (width 0) (type default) (color 0 0 0 0))
+  )
   (wire (pts (xy 207.01 157.48) (xy 218.44 157.48))
     (stroke (width 0) (type default) (color 0 0 0 0))
@@
     (stroke (width 0) (type default) (color 0 0 0 0))
   )
+  (polyline (pts (xy 342.9 95.25) (xy 342.9 139.7))
+    (stroke (width 0) (type default) (color 0 0 0 0))
+  )
   (polyline (pts (xy 76.2 13.97) (xy 76.2 116.84))
     (stroke (width 0) (type default) (color 0 0 0 0))
@@
     (stroke (width 0) (type default) (color 0 0 0 0))
   )
+  (wire (pts (xy 316.23 127) (xy 316.23 129.54))
+    (stroke (width 0) (type default) (color 0 0 0 0))
+  )
   (wire (pts (xy 201.93 62.23) (xy 201.93 63.5))
     (stroke (width 0) (type default) (color 0 0 0 0))
@@
     (stroke (width 0) (type default) (color 0 0 0 0))
   )
+  (polyline (pts (xy 267.97 95.25) (xy 267.97 139.7))
+    (stroke (width 0) (type default) (color 0 0 0 0))
+  )
   (wire (pts (xy 341.63 36.83) (xy 341.63 44.45))
     (stroke (width 0) (type default) (color 0 0 0 0))
@@
     (stroke (width 0) (type default) (color 0 0 0 0))
   )
+  (wire (pts (xy 316.23 104.14) (xy 316.23 106.68))
+    (stroke (width 0) (type default) (color 0 0 0 0))
+  )
   (wire (pts (xy 115.57 26.67) (xy 115.57 27.94))
     (stroke (width 0) (type default) (color 0 0 0 0))
@@
     (stroke (width 0) (type default) (color 0 0 0 0))
   )
+  (polyline (pts (xy 267.97 95.25) (xy 342.9 95.25))
+    (stroke (width 0) (type default) (color 0 0 0 0))
+  )
   (wire (pts (xy 314.96 44.45) (xy 314.96 46.99))
     (stroke (width 0) (type default) (color 0 0 0 0))
@@
   )
   (text "Power input" (at 342.9 60.96 0)
+    (effects (font (size 1.27 1.27)) (justify left bottom))
+  )
+  (text "RTC MODULE" (at 279.4 134.62 0)
     (effects (font (size 1.27 1.27)) (justify left bottom))
   )
@@
     )
   )
+  (global_label "SCL_RTC" (shape output) (at 138.43 69.85 0) (fields_autoplaced)
+    (effects (font (size 1.27 1.27)) (justify left))
+    (property "Intersheet References" "${INTERSHEET_REFS}" (id 0) (at 148.826 69.7706 0)
+      (effects (font (size 1.27 1.27)) (justify left) hide)
+    )
+  )
   (global_label "TXD" (shape input) (at 210.82 154.94 180) (fields_autoplaced)
     (effects (font (size 1.27 1.27)) (justify right))
@@
     )
   )
+  (global_label "SCL_RTC" (shape input) (at 298.45 111.76 180) (fields_autoplaced)
+    (effects (font (size 1.27 1.27)) (justify right))
+    (property "Intersheet References" "${INTERSHEET_REFS}" (id 0) (at 288.054 111.8394 0)
+      (effects (font (size 1.27 1.27)) (justify right) hide)
+    )
+  )
   (global_label "RESET" (shape input) (at 212.09 74.93 0) (fields_autoplaced)
     (effects (font (size 1.27 1.27)) (justify left))
@@
     )
   )
+  (global_label "SDA_RTC" (shape output) (at 137.16 67.31 0) (fields_autoplaced)
+    (effects (font (size 1.27 1.27)) (justify left))
+    (property "Intersheet References" "${INTERSHEET_REFS}" (id 0) (at 147.6164 67.2306 0)
+      (effects (font (size 1.27 1.27)) (justify left) hide)
+    )
+  )
   (global_label "TXD" (shape output) (at 133.35 82.55 0) (fields_autoplaced)
     (effects (font (size 1.27 1.27)) (justify left))
@@
     (effects (font (size 1.27 1.27)) (justify right))
     (property "Intersheet References" "${INTERSHEET_REFS}" (id 0) (at 202.1174 152.4794 0)
+      (effects (font (size 1.27 1.27)) (justify right) hide)
+    )
+  )
+  (global_label "SDA_RTC" (shape input) (at 288.29 114.3 180) (fields_autoplaced)
+    (effects (font (size 1.27 1.27)) (justify right))
+    (property "Intersheet References" "${INTERSHEET_REFS}" (id 0) (at 277.8336 114.2206 0)
       (effects (font (size 1.27 1.27)) (justify right) hide)
     )
@@
     (pin "9")
   )
+  (symbol (lib_id "HPS:VCC") (at 313.69 104.14 0) (unit 1)
+    (in_bom yes) (on_board yes) (fields_autoplaced)
+    (property "Reference" "#PWR?" (id 0) (at 313.69 107.95 0)
+      (effects (font (size 1.27 1.27)) hide)
+    )
+    (property "Value" "VCC" (id 1) (at 313.69 99.06 0))
+    (property "Footprint" "" (id 2) (at 313.69 104.14 0)
+      (effects (font (size 1.27 1.27)) hide)
+    )
+    (property "Datasheet" "" (id 3) (at 313.69 104.14 0)
+      (effects (font (size 1.27 1.27)) hide)
+    )
+    (pin "1")
+  )
+  (symbol (lib_id "HPS:GND") (at 316.23 129.54 0) (unit 1)
+    (in_bom yes) (on_board yes) (fields_autoplaced)
+    (property "Reference" "#PWR?" (id 0) (at 316.23 135.89 0)
+      (effects (font (size 1.27 1.27)) hide)
+    )
+    (property "Value" "GND" (id 1) (at 316.23 134.62 0))
+    (property "Footprint" "" (id 2) (at 316.23 129.54 0)
+      (effects (font (size 1.27 1.27)) hide)
+    )
+    (property "Datasheet" "" (id 3) (at 316.23 129.54 0)
+      (effects (font (size 1.27 1.27)) hide)
+    )
+    (pin "1")
+  )
+  (symbol (lib_id "HPS:+BATT") (at 316.23 104.14 0) (unit 1)
+    (in_bom yes) (on_board yes)
+    (property "Reference" "#PWR?" (id 0) (at 316.23 107.95 0)
+      (effects (font (size 1.27 1.27)) hide)
+    )
+    (property "Value" "+BATT" (id 1) (at 318.77 99.06 0))
+    (property "Footprint" "" (id 2) (at 316.23 104.14 0)
+      (effects (font (size 1.27 1.27)) hide)
+    )
+    (property "Datasheet" "" (id 3) (at 316.23 104.14 0)
+      (effects (font (size 1.27 1.27)) hide)
+    )
+    (pin "1")
+  )
   (symbol (lib_id "HPS:C_0805_22pf") (at 175.26 40.64 270) (unit 1)
     (in_bom yes) (on_board yes)
@@
     )
     (pin "1")
+  )
+  (symbol (lib_id "HPS:DS1307_DIP-8") (at 316.23 116.84 0) (unit 1)
+    (in_bom yes) (on_board yes) (fields_autoplaced)
+    (property "Reference" "U?" (id 0) (at 335.28 112.5093 0))
+    (property "Value" "DS1307_DIP-8" (id 1) (at 335.28 115.0493 0))
+    (property "Footprint" "footprints:DIP-8_W7.62mm" (id 2) (at 316.23 144.78 0)
+      (effects (font (size 1.27 1.27)) hide)
+    )
+    (property "Datasheet" "https://datasheets.maximintegrated.com/en/ds/DS1307.pdf" (id 3) (at 316.23 121.92 0)
+      (effects (font (size 1.27 1.27)) hide)
+    )
+    (property "MFG" "Assmann WSW Components" (id 4) (at 316.23 139.7 0)
+      (effects (font (size 1.27 1.27)) hide)
+    )
+    (property "MPN" "A 08-LC-TT" (id 5) (at 316.23 142.24 0)
+      (effects (font (size 1.27 1.27)) hide)
+    )
+    (property "Digikey PN" "AE9986-ND" (id 6) (at 316.23 147.32 0)
+      (effects (font (size 1.27 1.27)) hide)
+    )
+    (property "Mouser PN" "N/A" (id 7) (at 316.23 149.86 0)
+      (effects (font (size 1.27 1.27)) hide)
+    )
+    (pin "1")
+    (pin "2")
+    (pin "3")
+    (pin "4")
+    (pin "5")
+    (pin "6")
+    (pin "7")
+    (pin "8")
   )
   (symbol (lib_id "HPS:MountingHole") (at 25.4 186.69 0) (unit 1)
@@
       (reference "#PWR011") (unit 1) (value "VCC") (footprint "")
     )
+    (path "/7180da92-bb59-4176-9201-5715498db688"
+      (reference "#PWR?") (unit 1) (value "VCC") (footprint "")
+    )
+    (path "/838de597-8cac-4757-89f4-6abfac334526"
+      (reference "#PWR?") (unit 1) (value "GND") (footprint "")
+    )
+    (path "/96855650-123f-45aa-8354-ccb9326b3a68"
+      (reference "#PWR?") (unit 1) (value "+BATT") (footprint "")
+    )
     (path "/63fe69fa-19f2-4018-bfe2-85b6913817f2"
       (reference "C1") (unit 1) (value "CP (1uF)") (footprint "footprints:C_0805_2012Metric")
@@
       (reference "U2") (unit 1) (value "L7805_TO92") (footprint "footprints:TO-92_Inline")
     )
+    (path "/a8130c85-9178-412d-89fb-797deee35bdc"
+      (reference "U?") (unit 1) (value "DS1307_DIP-8") (footprint "footprints:DIP-8_W7.62mm")
+    )
     (path "/6442dc18-36db-40d9-883c-94941bf3bbe3"

Commit message: updated with pcb
Parts:
- added BT1: Battery_Cell, footprints:BatteryHolder_Keystone_106_1x20mm, symbol HPS:Battery_Cell
- added C8, C9: C_0805_0.1uf, footprints:C_0805_2012Metric, symbol HPS:C_0805_0.1uf
- added D2, D3, D4, D5, D6, D7, D8: LED_0805_GRN, footprints:LED_0805_2012Metric, symbol HPS:LED_0805_GRN
- added DS1: LED_Display_1001, footprints:Adafruit-1001-0-0-MFG, symbol HPS:LED_Display_1001
- added J3: Conn_02x03_Odd_Even, footprints:PinHeader_2x03_P2.54mm_Vertical, symbol HPS:Conn_02x03_Odd_Even
- added R10: R_0805_22K, footprints:R_0805_2012Metric, symbol HPS:R_0805_22K
- added R11, R12, R5, R6, R7, R8, R9: R_0805_10K, footprints:R_0805_2012Metric, symbol HPS:R_0805_10K
- added SW2, SW3, SW4, SW5: Omron_B3F_SPST, footprints:SW_SPST_Omron_B3FS-100xP, symbol HPS:Omron_B3F_SPST
- added U4: MAX7219, footprints:DIP-24_W7.62mm, symbol HPS:MAX7219
- added Y2: Crystal_32768Hz, footprints:Crystal_SMD_2Pin_3.2x1.5mm, symbol HPS:Crystal_32768Hz
- gave numbers to parts that had none: 1
Connections:
- net GND: now also BT1.2 (-), C8.2, C9.2, J3.6 (Pin_6), SW2.1 (A), SW2.2 (A), SW3.1 (A), SW3.2 (A), SW4.1 (A), SW4.2 (A), SW5.1 (A), SW5.2 (A), U4.4 (GND), U4.9 (GND)
- net LED_SCK: now also J3.3 (Pin_3)
- net RESET: now also J3.5 (Pin_5)
- net VCC: now also C8.1, C9.1, J3.2 (Pin_2), R10.1, R11.1, R12.1, R5.1, R6.1, R7.1, R8.1, R9.1, U4.19 (V+)
- net DISP_DATA: now reaches U1.11 (PD5)
- net DISP_DATA: now also U4.1 (DIN)
- net DISP_CLK: now reaches U1.12 (PD6)
- net DISP_CLK: now also U4.13 (CLK)
- net BTN_MIN: now reaches U1.13 (PD7)
- net BTN_MIN: now also R11.2, SW4.3 (B), SW4.4 (B)
- net BTN_DAY: now reaches U1.14 (PB0)
- net BTN_DAY: now also R12.2, SW5.3 (B), SW5.4 (B)
- net MOSI: now reaches U1.17 (PB3)
- net MOSI: now also J3.4 (Pin_4)
- net MISO: now reaches U1.18 (PB4)
- net MISO: now also J3.1 (Pin_1)
- net BTN_SETOPT: now reaches U1.4 (PD2)
- net BTN_SETOPT: now also R5.2, R6.2, R7.2, R8.2, SW2.3 (B), SW2.4 (B)
- net DISP_LOAD: now reaches U1.5 (PD3)
- net DISP_LOAD: now also U4.12 (LOAD)
- net BTN_HOUR: now reaches U1.6 (PD4)
- net BTN_HOUR: now also R9.2, SW3.3 (B), SW3.4 (B)
- net at U3.1 (X1): now also Y2.2
- net at U3.2 (X2): now also Y2.1
- net +BATT: no longer names the net of U3.3 (VBAT)
- net +BATT: now also BT1.1 (+)
- new net: D2.1 (K), D3.1 (K), D4.1 (K), D5.1 (K), D6.1 (K), D7.1 (K), D8.1 (K), U4.10 (DIG_5)
- new net: R10.2, U4.18 (ISET)
- new net DIG_0: DS1.14 (COM_DIG.1), U4.2 (DIG_0)
- new net DIG_1: DS1.11 (COM_DIG.2), U4.11 (DIG_1)
- new net DIG_2: DS1.10 (COM_DIG.3), U4.6 (DIG_2)
- new net DIG_3: DS1.6 (COM_DIG.4), U4.7 (DIG_3)
- new net DIG_4: DS1.7 (COM_COLON), U4.3 (DIG_4)
- new net SEG_A: D2.2 (A), DS1.13 (A), U4.14 (SEG_A)
- new net SEG_B: D3.2 (A), DS1.9 (B), U4.16 (SEG_B)
- new net SEG_C: D4.2 (A), DS1.4 (C), U4.20 (SEG_C)
- new net SEG_D: D5.2 (A), DS1.2 (D), U4.23 (SEG_D)
- new net SEG_DP: DS1.3 (DP), DS1.8 (COLON), U4.22 (SEG_DP)
- new net SEG_E: D6.2 (A), DS1.1 (E), U4.21 (SEG_E)
- new net SEG_F: D7.2 (A), DS1.12 (F), U4.15 (SEG_F)
- new net SEG_G: D8.2 (A), DS1.5 (G), U4.17 (SEG_G)
- no-connect marks 2 -> 12
Other:
- note added: "Buttons"
- note added: "ICSP"
- note added: "MAX_7219, 4_DIG_DISPLAY & 7 LED's"
- moved on the sheet: C1, C2, C3, C4, C5, C6, C7, J1, J2, R2, R3, R4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

Commit message: pcb routing
Parts:
- removed J2: PJ-102AH, footprints:PJ-102AH, symbol HPS:PJ-102AH
- removed R6, R7, R8: R_0805_10K, footprints:R_0805_2012Metric, symbol HPS:R_0805_10K
- added J2: Power_inlet_vertical, footprints:Wurth-694106402002, symbol HPS:Power_inlet_vertical
- added R13, R14: R_0805_4.7K, footprints:R_0805_2012Metric, symbol HPS:R_0805_4.7K
- U2: footprint footprints:TO-92_Inline -> footprints:TO-252-2
Connections:
- net GND: now also J2.2 (OUT)
- net SCL_RTC: now also R14.2
- net SDA_RTC: now also R13.2
- net VCC: now also R13.1, R14.1
- net at C1.1, U2.3 (VI): now also J2.1 (POLE)
- net DIG_5: now reaches D2.1 (K), D3.1 (K), D4.1 (K), D5.1 (K), D6.1 (K), D7.1 (K), D8.1 (K), U4.10 (DIG_5)
- net ISET: now reaches R10.2, U4.18 (ISET)

Commit message: new routing + gerber
Parts:
- removed U2: L7805_TO92, footprints:TO-252-2, symbol HPS:L7805_TO92
- added U2: L7805, footprints:TO-252-2, symbol HPS:L7805
Connections:
- net GND: now also U2.2 (GND)
- net VCC: now also U2.3 (OUT)
- net at C1.1, J2.1 (POLE): now also U2.1 (IN)

Commit message: final. I hope
Parts:
- added TP1, TP2, TP3, TP4, TP5, TP6, TP7: TestPoint, footprints:TestPoint_THTPad_D2.0mm_Drill1.0mm, symbol HPS:TestPoint
Connections:
- net DISP_CLK: now also TP7.1
- net DISP_DATA: now also TP6.1
- net DISP_LOAD: now also TP5.1
- net SCL_RTC: now also TP3.1
- net SDA_RTC: now also TP2.1
- net VCC: now also TP1.1
- net at BT1.1 (+), U3.3 (VBAT): now also TP4.1

Commit message: new changes
Parts:
- removed C1: CP (1uF), footprints:C_0805_2012Metric, symbol HPS:C_0805_10uf
- removed C4: C(0.1uF), footprints:C_0805_2012Metric, symbol HPS:C_0805_1uf
- removed C8: C_0805_0.1uf, footprints:C_0805_2012Metric, symbol HPS:C_0805_0.1uf
- removed R13, R14: R_0805_4.7K, footprints:R_0805_2012Metric, symbol HPS:R_0805_4.7K
- added C1: C_0805_1uf, footprints:C_0805_2012Metric, symbol HPS:C_0805_1uf
- added C4: C_0805_0.1uf, footprints:C_0805_2012Metric, symbol HPS:C_0805_0.1uf
- added C8: C_0805_10uf, footprints:C_0805_2012Metric, symbol HPS:C_0805_10uf
- added R6, R7: R_0805_4.7K, footprints:R_0805_2012Metric, symbol HPS:R_0805_4.7K
- C2: value C (0.1uF) -> C_0805_0.1uf
- C3, C5: value 22pf -> C_0805_22pf
- C7: value C(0.1uf) -> C_0805_0.1uf
- D1: value LED -> LED_0805
- R1: value 2.2K -> R_0805_2.2K
- R2: value 10K -> R_0805_10K
- Y1: value Crystal(16MHz) -> Crystal_32768Hz
Connections:
- net GND: now also C7.2, C1.2, C4.2, C8.2
- net SCL_RTC: now also U1.28 (SCL/PC5), R7.2; no longer U1.27 (SDA/PC4)
- net SDA_RTC: now also U1.27 (SDA/PC4), R6.2; no longer U1.26 (ADC3/PC3)
- net VCC: now also U1.20 (AVCC), U1.7 (VCC), C4.1, C8.1, R6.1, R7.1
- net at J2.1 (POLE), U2.1 (IN): now also C1.1
